File: ROBOT/_autosave-LSM6DOX.kicad_sch (KiCad schematic)
At the start: 7 parts

Commit message: update
Parts:
- U$1: footprint Adafruit_LSM6DSOX:LGA-14L -> Package_LGA:LGA-14_3x2.5mm_P0.5mm_LayoutBorder3x4y
Changed lines of the file:
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@@
 			)
 		)
-		(property "Footprint" "Adafruit_LSM6DSOX:LGA-14L"
+		(property "Footprint" "Package_LGA:LGA-14_3x2.5mm_P0.5mm_LayoutBorder3x4y"
 			(at 157.48 102.87 0)
 			(effects
