File: ROBOT/Robot.kicad_sch (KiCad schematic)
At the start: 14 parts, among them J1 Conn_02x20_Odd_Even, J2 MCP3208, J5 Battery

Commit message: update
Parts:
- C20: value 220uF -> 330uF
- J1: footprint Connector_PinHeader_2.54mm:PinHeader_2x20_P2.54mm_Vertical -> Connector_PinSocket_2.54mm:PinSocket_2x20_P2.54mm_Vertical
Changed lines of the file:
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@@
 			)
 		)
-		(property "Value" "220uF"
+		(property "Value" "330uF"
 			(at 45.466 56.388 0)
 			(effects
@@
 			)
 		)
-		(property "Footprint" "Connector_PinHeader_2.54mm:PinHeader_2x20_P2.54mm_Vertical"
+		(property "Footprint" "Connector_PinSocket_2.54mm:PinSocket_2x20_P2.54mm_Vertical"
 			(at 43.18 128.27 0)
 			(effects
