File: ROBOT/Robot.kicad_sch (KiCad schematic)
At the start: 14 parts, among them J1 Conn_02x20_Odd_Even, J2 MCP3208, J5 Battery

Commit message: update
Other:
- note added: "LEDD"
- note removed: "LED"
Changed lines of the file:
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@@
 		)
 	)
-	(text "LED\n\n"
+	(text "LEDD\n\n\n\n"
 		(exclude_from_sim no)
-		(at 76.962 84.328 0)
+		(at 76.962 86.614 0)
 		(effects
 			(font

Commit message: update pcb
Parts:
- C21: footprint Capacitor_SMD:C_0603_1608Metric_Pad1.08x0.95mm_HandSolder -> Capacitor_SMD:C_0805_2012Metric_Pad1.18x1.45mm_HandSolder
Changed lines of the file:
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@@
 			)
 		)
-		(property "Footprint" "Capacitor_SMD:C_0603_1608Metric_Pad1.08x0.95mm_HandSolder"
+		(property "Footprint" "Capacitor_SMD:C_0805_2012Metric_Pad1.18x1.45mm_HandSolder"
 			(at 53.34 55.88 0)
 			(effects
