File: ROBOT/LSM6DOX.kicad_sch (KiCad schematic)
At the start: 7 parts

Commit message: update
Parts:
- U$1: footprint Adafruit_LSM6DSOX:LGA-14L -> Package_LGA:LGA-14_3x2.5mm_P0.5mm_LayoutBorder3x4y
Changed lines of the file:
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@@
 			)
 		)
-		(property "Footprint" "Adafruit_LSM6DSOX:LGA-14L"
+		(property "Footprint" "Package_LGA:LGA-14_3x2.5mm_P0.5mm_LayoutBorder3x4y"
 			(at 157.48 102.87 0)
 			(effects

Commit message: First Routage
Parts:
- removed R17: 0, Resistor_SMD:R_0603_1608Metric_Pad0.98x0.95mm_HandSolder, symbol Device:R
Connections:
- net +3.3V: now also C12.2, C13.2, R18.1, R19.1, R20.1, U$1.5 (VDDIO), U$1.8 (VDD)
Changed lines of the file:
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@@
-	(wire
-		(pts
-			(xy 114.3 78.74) (xy 119.38 78.74)
-		)
-		(stroke
-			(width 0)
-			(type default)
-		)
-	)
 	(wire
 		(pts
@@
 	(wire
 		(pts
-			(xy 101.6 78.74) (xy 106.68 78.74)
+			(xy 101.6 78.74) (xy 119.38 78.74)
 		)
 		(stroke
@@
 					(unit 1)
 				)
-			)
-		)
-	)
-	(symbol
-		(lib_id "Device:R")
-		(at 110.49 78.74 270)
-		(unit 1)
-		(exclude_from_sim no)
-		(in_bom yes)
-		(on_board yes)
-		(dnp no)
-		(fields_autoplaced yes)
-		(property "Reference" "R17"
-			(at 110.49 72.39 90)
-			(effects
-				(font
-					(size 1.27 1.27)
-				)
-			)
-		)
-		(property "Value" "0"
-			(at 110.49 74.93 90)
-			(effects
-				(font
-					(size 1.27 1.27)
-				)
-			)
-		)
-		(property "Footprint" "Resistor_SMD:R_0603_1608Metric_Pad0.98x0.95mm_HandSolder"
-			(at 110.49 76.962 90)
-			(effects
-				(font
-					(size 1.27 1.27)
-				)
-				(hide yes)
-			)
-		)
-		(property "Datasheet" "~"
-			(at 110.49 78.74 0)
-			(effects
-				(font
-					(size 1.27 1.27)
-				)
-				(hide yes)
-			)
-		)
-		(property "Description" "Resistor"
-			(at 110.49 78.74 0)
-			(effects
-				(font
-					(size 1.27 1.27)
-				)
-				(hide yes)
-			)
-		)
-		(pin "2"
-		)
-		(pin "1"
-		)
-		(instances
-			(project "Robot"
-				(path "/f1dd5862-79ad-43be-9f5c-46baed2cd441/262830eb-cda8-481d-a25c-bbba49056e31"
-					(reference "R17")
-					(unit 1)
-				)
