File: ROBOT/_autosave-Robot.kicad_pcb (KiCad board)
At the start: 4 copper layers, 65 x 30 mm, 52 parts, among them J1 Conn_02x20_Odd_Even, J2 MCP3208, J3 Conn_01x04, J4 Conn_01x04, J5 Battery, U1 TMC2225-SA-T, U2 TMC2225-SA-T

Commit message: PCB 3D
Parts:
- moved C11 1.95 mm to (142.5, 100.5)
- moved C14 1.95 mm to (144.8, 100.5)
Routing:
- net GND: track 22.3 -> 39.8 mm, vias 17 -> 22
Changed lines of the file:
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@@
 	(footprint "Capacitor_SMD:C_0805_2012Metric_Pad1.18x1.45mm_HandSolder"
 		(layer "F.Cu")
-		(at 141 101.75 -90)
+		(at 142.5 100.5 -90)
 		(descr "Capacitor SMD 0805 (2012 Metric), square (rectangular) end terminal, IPC-7351 nominal with elongated pad for handsoldering. (Body size source: IPC-SM-782 page 76, https://www.pcb-3d.com/wordpress/wp-content/uploads/ipc-sm-782a_amendment_1_and_2.pdf, https://docs.google.com/spreadsheets/d/1BsfQQcO9C6DZCsRaXUlFlo91Tg2WpOkGARC1WS5S8t0/edit?usp=sharing), generated with kicad-footprint-generator")
 		(tags "capacitor handsolder")
@@
 	(footprint "Capacitor_SMD:C_0805_2012Metric_Pad1.18x1.45mm_HandSolder"
 		(layer "F.Cu")
-		(at 143.25 101.75 -90)
+		(at 144.75 100.5 -90)
 		(descr "Capacitor SMD 0805 (2012 Metric), square (rectangular) end terminal, IPC-7351 nominal with elongated pad for handsoldering. (Body size source: IPC-SM-782 page 76, https://www.pcb-3d.com/wordpress/wp-content/uploads/ipc-sm-782a_amendment_1_and_2.pdf, https://docs.google.com/spreadsheets/d/1BsfQQcO9C6DZCsRaXUlFlo91Tg2WpOkGARC1WS5S8t0/edit?usp=sharing), generated with kicad-footprint-generator")
 		(tags "capacitor handsolder")
@@
 	)
 	(segment
-		(start 142.75 99.25)
-		(end 143.25 99.75)
+		(start 144.25 98)
+		(end 144.75 98.5)
 		(width 0.2)
 		(layer "F.Cu")
@@
 	)
 	(segment
-		(start 142.25 99.25)
-		(end 141.75 99.25)
+		(start 143.75 98)
+		(end 143.25 98)
 		(width 0.2)
 		(layer "F.Cu")
@@
 	)
 	(segment
-		(start 141.75 99.25)
-		(end 141 100)
+		(start 143.25 98)
+		(end 142.5 98.75)
 		(width 0.2)
 		(layer "F.Cu")
@@
 	)
 	(segment
-		(start 142.25 99.25)
-		(end 142.75 99.25)
+		(start 143.75 98)
+		(end 144.25 98)
 		(width 0.2)
 		(layer "F.Cu")
@@
 	)
 	(segment
-		(start 141 100)
-		(end 141 100.7125)
+		(start 142.5 98.75)
+		(end 142.5 99.4625)
 		(width 0.2)
 		(layer "F.Cu")
@@
 	)
 	(segment
-		(start 143.25 99.75)
-		(end 143.25 100.7125)
+		(start 144.75 98.5)
+		(end 144.75 99.4625)
 		(width 0.2)
 		(layer "F.Cu")
@@
 	)
 	(via
-		(at 142.25 99.25)
+		(at 143.75 98)
 		(size 0.6)
 		(drill 0.3)
@@
 	)
 	(segment
+		(start 140.45 98.45)
+		(end 140.45 96.5)
+		(width 0.4)
+		(layer "F.Cu")
+		(net 2)
+	)
+	(segment
 		(start 174.475 94.5875)
 		(end 174.5125 94.55)
@@
 	)
 	(segment
+		(start 144 108)
+		(end 145.125 108)
+		(width 0.2)
+		(layer "F.Cu")
+		(net 2)
+	)
+	(segment
 		(start 172 86.5)
 		(end 172 87.6375)
@@
 	)
 	(segment
-		(start 139.5 102.5)
-		(end 140.7125 102.5)
+		(start 140.5 93.95)
+		(end 140.45 94)
+		(width 0.4)
+		(layer "F.Cu")
+		(net 2)
+	)
+	(segment
+		(start 145.125 108)
+		(end 145.25 108.125)
 		(width 0.2)
 		(layer "F.Cu")
@@
 	)
 	(segment
+		(start 141 101.25)
+		(end 142.2125 101.25)
+		(width 0.4)
+		(layer "F.Cu")
+		(net 2)
+	)
+	(segment
 		(start 156.5 87.5)
 		(end 156.5 88.8375)
@@
 	)
 	(segment
+		(start 155 103)
+		(end 155 105.8)
+		(width 0.2)
+		(layer "F.Cu")
+		(net 2)
+	)
+	(segment
 		(start 187.5 91.8)
 		(end 187.3 92)
@@
 	)
 	(segment
-		(start 140.7125 102.5)
-		(end 141 102.7875)
-		(width 0.2)
+		(start 142.2125 101.25)
+		(end 142.5 101.5375)
+		(width 0.4)
 		(layer "F.Cu")
 		(net 2)
@@
 	)
 	(segment
+		(start 140.5 92.5)
+		(end 140.5 93.95)
+		(width 0.4)
+		(layer "F.Cu")
+		(net 2)
+	)
+	(segment
 		(start 172.65 94.55)
 		(end 171.3 93.2)
@@
 	)
 	(segment
+		(start 152 108)
+		(end 150.625 108)
+		(width 0.2)
+		(layer "F.Cu")
+		(net 2)
+	)
+	(segment
 		(start 164.5 95.7125)
 		(end 165 95.7125)
@@
 	)
 	(segment
+		(start 174.5 99.1125)
+		(end 174.5125 99.1)
+		(width 0.2)
+		(layer "F.Cu")
+		(net 2)
+	)
+	(segment
 		(start 174 86)
 		(end 174 87.1375)
@@
 	)
 	(segment
+		(start 173.25 106.5)
+		(end 173.25 105.25)
+		(width 0.4)
+		(layer "F.Cu")
+		(net 2)
+	)
+	(segment
+		(start 144.5 101.7875)
+		(end 144.75 101.5375)
+		(width 0.2)
+		(layer "F.Cu")
+		(net 2)
+	)
+	(segment
+		(start 140.5 98.5)
+		(end 140.45 98.45)
+		(width 0.4)
+		(layer "F.Cu")
+		(net 2)
+	)
+	(segment
 		(start 187.5 90.5)
 		(end 187.5 91.8)
-		(width 0.2)
+		(width 0.4)
+		(layer "F.Cu")
+		(net 2)
+	)
+	(segment
+		(start 173.25 105.25)
+		(end 175 103.5)
+		(width 0.4)
 		(layer "F.Cu")
 		(net 2)
@@
 		(start 184.5 86)
 		(end 184.5 86.9625)
-		(width 0.2)
+		(width 0.4)
 		(layer "F.Cu")
 		(net 2)
@@
 	)
 	(segment
-		(start 143.5375 102.5)
-		(end 143.25 102.7875)
-		(width 0.2)
+		(start 145.0375 101.25)
+		(end 144.75 101.5375)
+		(width 0.4)
 		(layer "F.Cu")
 		(net 2)
@@
 		(start 188.5 98)
 		(end 188.5 96.55)
-		(width 0.2)
+		(width 0.4)
 		(layer "F.Cu")
 		(net 2)
@@
 	)
 	(segment
+		(start 150.625 108)
+		(end 150.5 108.125)
+		(width 0.2)
+		(layer "F.Cu")
+		(net 2)
+	)
+	(segment
 		(start 188.5 96.55)
 		(end 188.55 96.5)
@@
 	)
 	(segment
+		(start 150.5 108.125)
+		(end 148.75 108.125)
+		(width 0.2)
+		(layer "F.Cu")
+		(net 2)
+	)
+	(segment
 		(start 182 86)
 		(end 182 87.2125)
+		(width 0.4)
+		(layer "F.Cu")
+		(net 2)
+	)
+	(segment
+		(start 144.5 103)
+		(end 144.5 101.7875)
+		(width 0.4)
+		(layer "F.Cu")
+		(net 2)
+	)
+	(segment
+		(start 174.5 100)
+		(end 174.5 99.1125)
 		(width 0.2)
 		(layer "F.Cu")
@@
 	)
 	(segment
-		(start 145 102.5)
-		(end 143.5375 102.5)
+		(start 145.25 108.125)
+		(end 147 108.125)
 		(width 0.2)
 		(layer "F.Cu")
@@
 	)
 	(via
-		(at 139.5 102.5)
+		(at 175 103.5)
 		(size 0.6)
 		(drill 0.3)
@@
 	)
 	(via
-		(at 145 102.5)
+		(at 141 101.25)
 		(size 0.6)
 		(drill 0.3)
@@
 	)
 	(via
+		(at 155 103)
+		(size 0.6)
+		(drill 0.3)
+		(layers "F.Cu" "B.Cu")
+		(free yes)
+		(net 2)
+	)
+	(via
 		(at 184.5 86)
 		(size 0.6)
@@
 	)
 	(via
+		(at 144.5 103)
+		(size 0.6)
+		(drill 0.3)
+		(layers "F.Cu" "B.Cu")
+		(free yes)
+		(net 2)
+	)
+	(via
+		(at 152 108)
+		(size 0.6)
+		(drill 0.3)
+		(layers "F.Cu" "B.Cu")
+		(free yes)
+		(net 2)
+	)
+	(via
 		(at 187.5 90.5)
 		(size 0.6)
@@
 	)
 	(via
+		(at 144 108)
+		(size 0.6)
+		(drill 0.3)
+		(layers "F.Cu" "B.Cu")
+		(free yes)
+		(net 2)
+	)
+	(via
 		(at 165.6 96.7)
 		(size 0.6)
 		(drill 0.3)
+		(layers "F.Cu" "B.Cu")
+		(free yes)
+		(net 2)
+	)
+	(via
+		(at 174.5 100)
+		(size 0.6)
+		(drill 0.3)
