File: ROBOT/Robot.kicad_pcb (KiCad board)
At the start: 4 copper layers, 65 x 30 mm, 52 parts, among them J1 Conn_02x20_Odd_Even, J2 MCP3208, J3 Conn_01x04, J4 Conn_01x04, J5 Battery, U1 TMC2225-SA-T, U2 TMC2225-SA-T

Commit message: Update netclass
Parts:
- moved C11 1.95 mm to (142.5, 100.5)
- moved C14 1.95 mm to (144.8, 100.5)
- moved R6 1.77 mm to (187.0, 96.5)
- moved R11 1.46 mm to (142.0, 94.0)
- moved R13 1.46 mm to (142.0, 96.5)
- moved C5 1.12 mm to (144.5, 90.5)
- moved R8 0.50 mm to (185.8, 92.0)
Routing:
- net GND: track 9.65 -> 39.8 mm, vias 4 -> 22
- net VCC: track 32.9 -> 37.3 mm
- net Net-(D2-A): track 33.4 -> 35.9 mm, vias 2 -> 4
- net Net-(U1-VCP): track 2.64 -> 3.85 mm
- net Net-(D1-A): track 15.6 -> 16.8 mm, vias 2 -> 0
- net Net-(U2-BRA): track 4.42 -> 5.48 mm
- net Net-(U1-BRA): track 4.72 -> 5.66 mm
- net Net-(U1-BRB): track 5.54 -> 6.20 mm

Commit message: Update Robot.kicad_pcb
Parts:
- added C10: 10uF, Capacitor_SMD:C_0805_2012Metric_Pad1.18x1.45mm_HandSolder, F.Cu at (140.5, 100.5)
- added C9: 10uF, Capacitor_SMD:C_0805_2012Metric_Pad1.18x1.45mm_HandSolder, F.Cu at (186.5, 88.0)
- moved R8 0.50 mm to (185.8, 92.5)
Routing:
- net VCC: track 37.3 -> 44.6 mm
- net GND: track 39.8 -> 41.0 mm, vias 22 -> 23

Commit message: update PCB
Parts:
- C11, C14: footprint Capacitor_SMD:C_0805_2012Metric_Pad1.18x1.45mm_HandSolder -> Capacitor_SMD:C_0603_1608Metric_Pad1.08x0.95mm_HandSolder
- moved C11 10.0 mm to (142.0, 90.5), turned to 90 degrees
- moved C10 4.03 mm to (144.5, 100.0)
- moved C14 2.66 mm to (146.5, 98.5)
Routing:
- net VCC: track 44.6 -> 39.7 mm, vias 11 -> 10
- net GND: track 41.0 -> 39.4 mm

Commit message: Revue de shcema
Parts:
- C1, C2: footprint Capacitor_SMD:C_0805_2012Metric_Pad1.18x1.45mm_HandSolder -> Capacitor_SMD:C_0603_1608Metric_Pad1.08x0.95mm_HandSolder
- moved C2 11.4 mm to (186.0, 99.5), turned to -90 degrees
- moved C9 2.55 mm to (184.0, 88.5)
- moved C3 1.03 mm to (184.5, 100.0), turned to -90 degrees
Routing:
- net +3.3V: track 37.7 -> 32.8 mm
- net VCC: track 39.7 -> 37.1 mm
- net Net-(U2-VCP): track 3.43 -> 5.91 mm
- net Net-(U1-MS2): track 5.78 -> 3.64 mm
- net Net-(J4-Pin_4): track 14.9 -> 14.2 mm
- net GND: track 39.4 -> 39.6 mm, vias 23 -> 24
